File: CAD/Methanesense/Methanesense.kicad_pcb (KiCad board)
At the start: 4 copper layers, 120.3 x 25.6 mm, 92 parts, among them J1 USB_C_Receptacle_USB2.0_14P, J2 HIROSE ELECTRIC U.FL-R-SMT-1, J3 693043020611, J4 HIROSE ELECTRIC U.FL-R-SMT-1, J5 Conn_01x10_Pin, J6 JLINK, Q1 FDS6898A, Q2 FDS6898A, SW1 KMR223NGLFG, SW3 KMR223NGLFG, SW4 JS202011JCQN, U2 ADS1115IDGS, U3 nPM1300-QEXX, U4 AP7331-20WG-7, U5 nRF9160-SICA, U6 BME680, U7 FT230XQ, U8 USBLC6-4SC6, U9 TPS22917DBV

Commit message: Rev 2.0.0
Parts:
- added C15: 4.7uF, Capacitor_SMD:C_0603_1608Metric, F.Cu at (70.4, 65.9)
- added C16: 1uF, Capacitor_SMD:C_0603_1608Metric, F.Cu at (71.4, 68.2)
- added G***: LOGO, LOGO, F.Cu at (111.1, 59.7)
- U3: footprint Methanesense:QFN-32-1EP_5x5mm_P0.5mm_EP3.6x3.6mm -> Methanesense:QFN-32-1EP_5x5mm_P0.5mm_EP3.6x3.6mm_ThermalVias
- U5: footprint PCM_nordic-lib-kicad-nrf9:LGA_9160_16.0x10.5mm -> Methanesense:LGA_9160_16.0x10.5mm
- moved C11 1.62 mm to (71.4, 69.7)
- moved U8 1.49 mm to (63.6, 58.3)
- moved C31 1.31 mm to (66.9, 55.1), turned to 180 degrees
- moved C34 1.06 mm to (62.2, 54.8)
- moved J3 1.00 mm to (75.8, 55.5)
- moved R18 1.00 mm to (66.9, 56.6)
- moved R19 1.00 mm to (66.9, 58.1)
- moved R20 1.00 mm to (66.9, 59.6)
- moved C32 0.87 mm to (47.2, 54.4)
- moved J6 0.80 mm to (47.0, 61.8)
- moved C21 0.80 mm to (46.6, 52.0)
- moved U5 0.80 mm to (54.5, 60.8)
- moved C35 0.73 mm to (61.0, 54.4)
- moved C33 0.70 mm to (46.1, 54.3)
- moved C22 0.63 mm to (63.8, 54.5)
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Connections:
- D10 pad 2: +5V -> VSYS
- D11 pad 2: +5V -> VSYS
- D9 pad 2: +5V -> VSYS
- J5 pad 10: P0.08 -> P0.11
- J6 pad 3: unconnected-(J6-Pin_3-Pad3)_0 -> GND
- J6 pad 5: unconnected-(J6-Pin_5-Pad5) -> GND
- J6 pad 7: unconnected-(J6-Pin_7-Pad7) -> GND
- J6 pad 8: unconnected-(J6-Pin_8-Pad8) -> GND
- Q1 pad 2: P0.29 -> P0.27
- Q2 pad 2: P0.07 -> P0.06
- R11 pad 2: P0.29 -> P0.27
- R25 pad 2: P0.07 -> P0.06
- SW1 pad 1: P0.06 -> P0.07
- SW4 pad 2: P0.08 -> P0.11
- U2 pad 10: P0.27 -> P0.29
- U2 pad 2: P0.28 -> P0.26
- U2 pad 9: P0.26 -> P0.28
- U3 pad 13: P0.26 -> P0.28
- U3 pad 14: P0.27 -> P0.29
- U3 pad 32: +5V -> VSYS
- U6 pad 3: P0.26 -> P0.28
- U6 pad 4: P0.27 -> P0.29
- U7 pad 15: P0.11 -> P0.12
Routing:
- net P0.12: track 0.00 -> 90.9 mm, vias 0 -> 2
- net P0.08: track 87.6 -> 0.00 mm, vias 2 -> 0
- net GND: track 266.1 -> 351.5 mm, vias 403 -> 441
- net P0.27: track 122.4 -> 69.9 mm, vias 4 -> 2
- net P0.29: track 68.1 -> 117.1 mm, vias 2 -> 4
- net P0.26: track 120.8 -> 88.2 mm, vias 4 -> 2
- net P0.28: track 86.5 -> 114.3 mm, vias 2 -> 4
- net VSYS: track 13.1 -> 31.7 mm, vias 4 -> 6
- net +5V: track 141.5 -> 127.9 mm, vias 9 -> 8
- net SIM_RST: track 29.1 -> 36.5 mm
- net ~{RESET}: track 1.46 -> 8.32 mm
- net P0.11: track 86.3 -> 91.6 mm
- net +1V8SIM: track 37.2 -> 33.3 mm
- net P0.05: track 83.8 -> 80.1 mm
- net P0.19/AIN6: track 95.4 -> 97.8 mm
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- added copper zone on F.Cu, net +BATT
Other:
- outline, holes or cut-outs redrawn

Commit message: rev 1.2
Parts:
- removed AE1: NN02-220, Methanesense:XCVR_NN02-220
- removed C19: 0.1uF, Capacitor_SMD:C_0603_1608Metric
- removed C3: 47pF, Capacitor_SMD:C_0603_1608Metric
- removed C8, C9: 1uF, Capacitor_SMD:C_0603_1608Metric
- removed L4: NP, Methanesense:L_0603_1608Metric
- removed L5: 7.5NH, Methanesense:L_0603_1608Metric
- removed L6: 1.6nH, Methanesense:L_0603_1608Metric
- removed L7: 39NH, Methanesense:C_0402_1005Metric_Sqr
- removed SW4: JS202011JCQN, Button_Switch_SMD:SW_DPDT_CK_JS202011JCQN
- removed U4: AP7331-20WG-7, Package_TO_SOT_SMD:SOT-23-5
- removed U7: FT230XQ, Methanesense:QFN-16-1EP_4x4mm_P0.65mm_EP2.1x2.1mm
- added D1: D_scht, Diode_SMD:D_MicroSMP_AK, F.Cu at (124.2, 50.8)
- added D2: D_scht, Diode_SMD:D_MicroSMP_AK, F.Cu at (129.0, 56.8)
- added D3: D_scht, Diode_SMD:D_0603_1608Metric, F.Cu at (129.5, 64.5)
- added D4: D_scht, Diode_SMD:D_0603_1608Metric, F.Cu at (129.5, 66.2)
- added R12: 470R, Resistor_SMD:R_0603_1608Metric, F.Cu at (123.2, 69.5)
- added R13: 54.9k, Resistor_SMD:R_0603_1608Metric, F.Cu at (122.3, 57.5)
- added R14: 10k, Resistor_SMD:R_0603_1608Metric, F.Cu at (121.2, 55.2)
- added R15: 15k, Resistor_SMD:R_0603_1608Metric, F.Cu at (130.8, 50.0)
- added R16: 10k, Resistor_SMD:R_0603_1608Metric, F.Cu at (130.8, 48.5)
- added R21: 0R, Resistor_SMD:R_0603_1608Metric, F.Cu at (124.8, 65.5)
- added R27: 0R, Resistor_SMD:R_0603_1608Metric, F.Cu at (124.8, 60.5)
- added R28: 0R, Resistor_SMD:R_0603_1608Metric, F.Cu at (126.2, 60.5)
- added R30: 0R, Resistor_SMD:R_0603_1608Metric, F.Cu at (127.2, 65.5)
- added R37: 0R, Resistor_SMD:R_0603_1608Metric, F.Cu at (128.0, 50.0)
- added R6: 0R, Resistor_SMD:R_0603_1608Metric, F.Cu at (73.0, 73.0)
- added U1: LV2862XDDC, Package_TO_SOT_SMD:SOT-23-6, F.Cu at (124.6, 55.0)
- C1, C2: value 1.7pF -> 0.1uF; footprint Methanesense:C_0603_1608Metric -> Capacitor_SMD:C_0603_1608Metric
- C4: value 8.5pF -> 0.1uF; footprint Methanesense:C_0603_1608Metric -> Capacitor_SMD:C_0603_1608Metric
- C5: value 15pF -> 4.7uF; footprint Methanesense:C_0402_1005Metric_Sqr -> Capacitor_SMD:C_0603_1608Metric
- C6: value 47pF -> 4.7uF
- C7: value 1uF -> 4.7uF
- D5, D6: value LED -> D_scht; footprint LED_SMD:LED_0603_1608Metric -> Diode_SMD:D_0603_1608Metric
- J1: value USB_C_Receptacle_USB2.0_14P -> HIROSE ELECTRIC U.FL-R-SMT-1; footprint Methanesense:USB_C_Receptacle_HCTL_HC-TYPE-C-16P-01A -> Methanesense:U.FL_Hirose_U.FL-R-SMT-1_Vertical
- J2: value HIROSE ELECTRIC U.FL-R-SMT-1 -> IEC61076-2_M8_A-coding_01x04_Receptacle_Shielded; footprint Methanesense:U.FL_Hirose_U.FL-R-SMT-1_Vertical -> Methanesense:STEWART_SS-12800-004_M8_04_Socket_Right_Angle; moved to B.Cu
- J5: value Conn_01x10_Pin -> Conn_01x12_Pin; footprint Connector_PinHeader_2.54mm:PinHeader_1x10_P2.54mm_Vertical -> Connector_PinHeader_2.54mm:PinHeader_1x12_P2.54mm_Vertical; moved to B.Cu
- J6: moved to F.Cu
- L1: value 2.3nH -> 22uH; footprint Methanesense:L_0603_1608Metric -> Methanesense:L_Abracon_AMDLA4020S
- L8: value 68 nH -> 68 nH
- R22: value 100R -> 0R
- R23: value 100R -> 10k
- R26: value 1k -> 0R
- R4, R8: value 0R -> 1k
- R5: value 0R -> 470R
- R9: value <2k -> 12k
- moved J2 95.8 mm to (143.6, 60.8), turned to 90 degrees
- moved J1 83.8 mm to (65.4, 73.0), turned to 180 degrees
- moved C5 82.5 mm to (134.5, 54.5), turned to -90 degrees
- moved C4 79.8 mm to (124.5, 52.5), turned to 0 degrees
- moved L1 79.3 mm to (129.2, 53.2), turned to 0 degrees
- moved C2 69.4 mm to (120.2, 69.5), turned to 0 degrees
- moved C1 65.2 mm to (120.2, 68.0), turned to 0 degrees
- moved R4 54.2 mm to (132.5, 64.5), turned to 180 degrees
- moved R23 38.4 mm to (132.5, 66.0), turned to 180 degrees
- moved D5 35.8 mm to (130.0, 59.8), turned to 180 degrees
- moved D6 31.5 mm to (130.0, 61.2), turned to 180 degrees
- moved R22 30.7 mm to (126.0, 65.5), turned to 90 degrees
- moved U8 26.1 mm to (89.2, 63.0), turned to 180 degrees
- moved R26 25.7 mm to (127.8, 60.5), turned to 90 degrees
- moved J4 25.4 mm to (88.2, 73.0)
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Connections:
- net /nrf9160/GPS renamed Net-(U5-GPS)
- C1 pad 1: Net-(C1-Pad1) -> GND
- C1 pad 2: Net-(C1-Pad2) -> /GAS_SENSOR/AIN2_
- C12 pad 1: VSYS -> VCC
- C2 pad 1: Net-(C2-Pad1) -> GND
- C2 pad 2: GND -> /GAS_SENSOR/AIN3_
- C20 pad 1: +2V0SW -> +2V0
- C21 pad 1: +5V -> VCC
- C22 pad 1: +5V -> VCC
- C24 pad 1: +5V -> VCC
- C27 pad 2: Net-(C1-Pad1) -> Net-(C27-Pad2)
- C28 pad 1: +5V -> VCC
- C32 pad 1: +5V -> VCC
- C33 pad 1: +5V -> VCC
- C34 pad 1: +5V -> VCC
- C35 pad 1: +5V -> VCC
- C37 pad 1: VSYS -> VCC
- C38 pad 1: +2V0SW -> +2V0
- C39 pad 1: +2V0SW -> +2V0
- C4 pad 1: Net-(C2-Pad1) -> Net-(U1-CB)
- C4 pad 2: Net-(C4-Pad2) -> /POWER/SW
- C5 pad 1: /nrf9160/ANT -> /POWER/SW5V
- C5 pad 2: Net-(J2-In) -> GND
- C6 pad 1: GND -> /POWER/SW5V
- C6 pad 2: /POWER/USBDP -> GND
- C7 pad 1: /POWER/VCCIOUSB -> /POWER/SW5V
- D10 pad 2: VSYS -> VCC
- D11 pad 2: VSYS -> VCC
- D5 pad 1: Net-(D5-K) -> +2V0
- D6 pad 1: Net-(D6-K) -> Net-(D5-A)
- D6 pad 2: Net-(D6-A) -> GND
- D9 pad 2: VSYS -> VCC
- J2 pad 1: Net-(J2-In) -> /POWER/VIN
- J2 pad 2: GND -> /POWER/GPIO1
- J5 pad 1: +2V0 -> GND
- J5 pad 10: P0.11 -> P0.19/AIN6
- J5 pad 2: +5V -> +BATT
- J5 pad 3: +BATT -> GND
- J5 pad 4: GND -> +2V0
- J5 pad 5: +5VL -> GND
- J5 pad 6: GND -> P0.08
- J5 pad 7: P0.07 -> P0.09
- J5 pad 8: P0.06 -> P0.10
- J5 pad 9: P0.05 -> P0.18/AIN5
- L1 pad 1: Net-(C1-Pad2) -> /POWER/SW
- L1 pad 2: Net-(C2-Pad1) -> /POWER/SW5V
- L2 pad 1: Net-(C1-Pad1) -> Net-(C27-Pad2)
- Q2 pad 2: P0.06 -> P0.17/AIN4
- Q2 pad 4: P0.05 -> P0.01
- Q2 pad 5: Net-(D6-K) -> /POWER/OD1
- Q2 pad 6: Net-(D6-K) -> /POWER/OD1
- Q2 pad 7: Net-(D5-K) -> /POWER/OD2
- Q2 pad 8: Net-(D5-K) -> /POWER/OD2
- R22 pad 1: +2V0 -> P0.16/AIN3
- R22 pad 2: Net-(D6-A) -> Net-(D3-K)
- R23 pad 1: Net-(D5-A) -> /POWER/GPIO1
- R23 pad 2: +2V0 -> Net-(D3-K)
- R24 pad 2: P0.05 -> P0.01
- R25 pad 2: P0.06 -> P0.17/AIN4
- R26 pad 1: GND -> /GAS_SENSOR/AIN3
- R26 pad 2: Net-(SW4A-A) -> Net-(D5-A)
- R4 pad 1: +2V0 -> GND
- R4 pad 2: +2V0SW -> Net-(D3-K)
- R5 pad 1: P0.04 -> /GAS_SENSOR/AIN2_
- R5 pad 2: /POWER/VCCIOUSB -> /GAS_SENSOR/AIN2
- R7 pad 1: P0.19/AIN6 -> /POWER/GPIO2
- R7 pad 2: /GAS_SENSOR/AIN0_ -> Net-(D5-A)
- R8 pad 1: /GAS_SENSOR/AIN1_ -> GND
- R8 pad 2: P0.18/AIN5 -> Net-(D5-A)
- S1 pad 3: +2V0SW -> +2V0
- S1 pad 4: +2V0SW -> +2V0
- SW1 pad 1: P0.07 -> P0.04
- U2 pad 6: AIN2 -> /GAS_SENSOR/AIN2_
- U2 pad 7: AIN3 -> /GAS_SENSOR/AIN3_
- U2 pad 8: +2V0SW -> +2V0
- U3 pad 20: VSYS -> VCC
- U3 pad 32: VSYS -> VCC
- U3 pad 4: VSYS -> VCC
- U3 pad 8: unconnected-(U3-GPIO1-Pad8) -> P0.11
- U3 pad 9: unconnected-(U3-GPIO2-Pad9) -> P0.12
- U5 pad 101: +5V -> VCC
- U5 pad 102: +5V -> VCC
- U5 pad 22: +5V -> VCC
- U6 pad 2: +2V0SW -> +2V0
- U6 pad 6: +2V0SW -> +2V0
- U6 pad 8: +2V0SW -> +2V0
- U9 pad 1: +5V -> VCC
Routing:
- net +2V0SW: track 130.0 -> 0.00 mm, vias 4 -> 0
- net +5V: track 127.9 -> 3.12 mm, vias 8 -> 0
- net VCC: track 0.00 -> 98.3 mm, vias 0 -> 14
- net /POWER/CC2: track 89.9 -> 0.00 mm, vias 2 -> 0
- net /POWER/CC1: track 89.8 -> 0.00 mm, vias 2 -> 0
- net +5VL: track 150.2 -> 60.7 mm, vias 7 -> 5
- net P0.07: track 79.3 -> 1.60 mm, vias 2 -> 0
- net P0.06: track 78.6 -> 3.83 mm, vias 2 -> 0
- net GND: track 351.5 -> 285.0 mm, vias 441 -> 267
- net P0.17/AIN4: track 0.00 -> 48.4 mm, vias 0 -> 2
- net P0.19/AIN6: track 97.8 -> 52.8 mm, vias 2 -> 0
- net P0.14/AIN1: track 88.7 -> 44.1 mm
- net P0.18/AIN5: track 90.5 -> 49.4 mm, vias 2 -> 0
- net P0.16/AIN3: track 102.5 -> 62.0 mm, vias 4 -> 2
- net P0.12: track 90.9 -> 50.6 mm
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- added copper zone on In2.Cu, net +BATT
- added copper zone on F.Cu, net /POWER/SW
- added copper zone on F.Cu, net /POWER/SW5V
- added copper zone on B.Cu, net VCC
- added copper zone on F.Cu, net VCC
- added copper zone on In2.Cu, net VCC
- removed copper zone on B.Cu, net +2V0SW
- removed copper zone on F.Cu, net +2V0SW
- removed copper zone on F.Cu, net +5V
- removed copper zone on In2.Cu, net +5V
- removed copper zone on B.Cu, net VSYS
- removed copper zone on F.Cu, net VSYS
Other:
- board size 120.3 x 25.6 mm -> 91 x 30 mm
- board text added: "2V0"
- board text added: "GND"
- board text added: "LTE-M"
- board text added: "P08"
- board text added: "P09"
- board text added: "P10"
- board text added: "P14"
- board text added: "P18"
- board text added: "P19"
- board text added: "VBAT"
- board text removed: "LTE"
- board text removed: "MINA-MethaneSense Rev 2.0"

Commit message: Feat: Rev 1.3
Parts:
- added C8: 2.2uF, Capacitor_SMD:C_0805_2012Metric, F.Cu at (128.7, 58.6)
- added D7: LG L29K-G2J1-24-Z, LED_SMD:LED_0603_1608Metric, F.Cu at (87.4, 51.6)
- added D8: MSS1P3L-M3/89A, Diode_SMD:D_MicroSMP_AK, F.Cu at (119.4, 55.0)
- added H1: MountingHole, MountingHole:MountingHole_2.2mm_M2, F.Cu at (93.8, 74.4)
- added H2: MountingHole, MountingHole:MountingHole_2.2mm_M2, F.Cu at (117.8, 49.0)
- added R29: 150R, Resistor_SMD:R_0603_1608Metric, F.Cu at (84.0, 51.6)
- added R31: 0R, Resistor_SMD:R_0402_1005Metric, F.Cu at (72.6, 72.5)
- added R32: 0R, Resistor_SMD:R_0402_1005Metric, F.Cu at (69.4, 72.5)
- added R33: 0R, Resistor_SMD:R_0402_1005Metric, F.Cu at (71.0, 73.0)
- added R34: 0R, Resistor_SMD:R_0603_1608Metric, F.Cu at (124.7, 61.2)
- added TP1: SWDIO, TestPoint:TestPoint_Pad_D1.0mm, F.Cu at (69.5, 60.2)
- added TP10: I1, TestPoint:TestPoint_Pad_D1.0mm, F.Cu at (102.8, 71.8)
- added TP11: AIN1, TestPoint:TestPoint_Pad_D1.0mm, F.Cu at (141.0, 70.2)
- added TP12: AIN0, TestPoint:TestPoint_Pad_D1.0mm, F.Cu at (131.8, 74.5)
- added TP13: SEN, TestPoint:TestPoint_Pad_D1.0mm, F.Cu at (110.5, 75.0)
- added TP14: HEAT, TestPoint:TestPoint_Pad_D1.0mm, F.Cu at (110.2, 66.8)
- added TP15: GND, TestPoint:TestPoint_Pad_D1.0mm, F.Cu at (61.6, 58.2)
- added TP16: GND, TestPoint:TestPoint_Pad_D1.0mm, F.Cu at (119.4, 59.0)
- added TP17: GND, TestPoint:TestPoint_Pad_D1.0mm, F.Cu at (98.0, 75.6)
- added TP18: GND, TestPoint:TestPoint_Pad_D1.0mm, F.Cu at (148.1, 67.6)
- added TP2: SWDCLK, TestPoint:TestPoint_Pad_D1.0mm, F.Cu at (68.0, 57.5)
- added TP3: SWO, TestPoint:TestPoint_Pad_D1.0mm, F.Cu at (64.5, 56.8)
- added TP4: RST, TestPoint:TestPoint_Pad_D1.0mm, F.Cu at (69.8, 58.6)
- added TP5: VIN, TestPoint:TestPoint_Pad_D1.0mm, F.Cu at (139.2, 55.8)
- added TP6: IO1, TestPoint:TestPoint_Pad_D1.0mm, F.Cu at (123.0, 64.2)
- added TP7: IO2, TestPoint:TestPoint_Pad_D1.0mm, F.Cu at (125.8, 58.6)
- added TP8: 5V, TestPoint:TestPoint_Pad_D1.0mm, F.Cu at (135.2, 52.0)
- added TP9: 2V, TestPoint:TestPoint_Pad_D1.0mm, F.Cu at (105.5, 73.5)
- added kibuzzard-680A1FD4: G***, kibuzzard-680A1FD4, B.Cu at (120.4, 74.4)
- added kibuzzard-680B6FC7: G***, kibuzzard-680B6FC7, F.Cu at (137.2, 55.8)
- added kibuzzard-680B701D: G***, kibuzzard-680B701D, F.Cu at (136.7, 52.0)
- added kibuzzard-680B70A9: G***, kibuzzard-680B70A9, F.Cu at (141.0, 72.3)
- added kibuzzard-680B70C8: G***, kibuzzard-680B70C8, F.Cu at (129.6, 74.5)
- added kibuzzard-680B70F6: G***, kibuzzard-680B70F6, F.Cu at (112.0, 75.0)
- added kibuzzard-680B712B: G***, kibuzzard-680B712B, F.Cu at (111.8, 66.8)
- added kibuzzard-680B714A: G***, kibuzzard-680B714A, F.Cu at (107.0, 73.5)
- added kibuzzard-680B715D: G***, kibuzzard-680B715D, F.Cu at (102.7, 73.8)
- added kibuzzard-680B71B4: G***, kibuzzard-680B71B4, F.Cu at (121.2, 59.0)
- added kibuzzard-680B7297: G***, kibuzzard-680B7297, F.Cu at (122.3, 63.0)
- added kibuzzard-680B72A0: G***, kibuzzard-680B72A0, F.Cu at (124.1, 58.6)
- added kibuzzard-680B72CB: G***, kibuzzard-680B72CB, F.Cu at (66.5, 57.5)
- added kibuzzard-680B72EC: G***, kibuzzard-680B72EC, F.Cu at (68.0, 58.7)
- added kibuzzard-680B7325: G***, kibuzzard-680B7325, F.Cu at (71.0, 60.3)
- added kibuzzard-680B73BF: G***, kibuzzard-680B73BF, F.Cu at (62.7, 56.8)
- added kibuzzard-680B73D9: G***, kibuzzard-680B73D9, F.Cu at (63.4, 58.2)
- D1, D2: value D_scht -> MSS1P3L-M3/89A
- D3, D4, D5, D6: value D_scht -> SD0603S040S0R2
- J5: value Conn_01x12_Pin -> Conn_01x13_Pin; footprint Connector_PinHeader_2.54mm:PinHeader_1x12_P2.54mm_Vertical -> Connector_PinHeader_2.54mm:PinHeader_1x13_P2.54mm_Vertical
- R13: value 54.9k -> 56k
- R6: footprint Resistor_SMD:R_0603_1608Metric -> Resistor_SMD:R_0402_1005Metric
- U2: value ADS1115IDGS -> ADS1115IDGST
- moved R8 2.20 mm to (133.0, 62.0)
- moved R27 1.70 mm to (123.2, 61.2)
- moved R6 1.60 mm to (74.6, 73.0)
- moved J5 1.00 mm to (83.2, 49.2)
- moved R7 0.80 mm to (133.0, 60.5)
- moved D5 0.70 mm to (130.0, 60.5)
- moved D6 0.70 mm to (130.0, 62.0)
- moved R26 0.70 mm to (127.8, 61.2)
- moved R28 0.70 mm to (126.2, 61.2)
- moved L2 0.60 mm to (76.4, 72.5)
- moved SW1 0.38 mm to (108.8, 62.1)
- moved BT1 0.15 mm to (64.7, 62.0)
Connections:
- net Net-(D2-K) renamed +12V
- J2 pad 2: /POWER/GPIO1 -> /POWER/GPIO2
- J2 pad 4: /POWER/GPIO2 -> /POWER/GPIO1
- R6 pad 1: Net-(J1-In) -> Net-(R31-Pad1)
Routing:
- net +2V0SW: track 0.00 -> 28.7 mm, vias 0 -> 3
- net P0.04: track 56.6 -> 39.6 mm
- net +12V: track 3.59 -> 17.2 mm
- net /nrf9160/12vin: track 0.00 -> 9.82 mm
- net Net-(U3-SHPHLD): track 1.83 -> 8.21 mm
- net GND: track 285.0 -> 289.9 mm, vias 267 -> 384
- net /POWER/VIN: track 20.6 -> 16.4 mm
- net P0.31: track 39.0 -> 42.2 mm
- net P0.11: track 55.0 -> 52.4 mm
- net Net-(R31-Pad1): track 0.00 -> 2.58 mm
- net Net-(D5-A): track 9.58 -> 12.1 mm
- net P0.20/AIN7: track 2.51 -> 0.00 mm, vias 1 -> 0
- net /POWER/SW5V: track 12.1 -> 14.5 mm
- net Net-(J1-In): track 1.72 -> 4.04 mm
- net P0.27: track 42.6 -> 44.7 mm
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- added copper zone on In2.Cu, net +5VL
Other:
- outline, holes or cut-outs redrawn
- board text added: "100% NON ALIEN TECH MADE WITH LOVE AND TERRAN MATERIALS BY EARTHLINGS AT AD ${CURRENT_DATE}"
- board text added: "12V"
- board text added: "NEG"
- board text added: "POS"
