File: CAD/Methanesense/Methanesense.kicad_pcb (KiCad board)
At the start: 4 copper layers, 91 x 30 mm, 144 parts, among them J1 HIROSE ELECTRIC U.FL-R-SMT-1, J2 IEC61076-2_M8_A-coding_01x04_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, J3 693043020611, J4 HIROSE ELECTRIC U.FL-R-SMT-1, J5 Conn_01x13_Pin, J6 JLINK, Q1 FDS6898A, Q2 FDS6898A, SW1 KMR223NGLFG, SW3 KMR223NGLFG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

Commit message: Feat: Prettified repo Readme
Parts:
- added kibuzzard-680B71B4: G***, kibuzzard-680B71B4, F.Cu at (146.3, 67.6)
Routing:
- net GND: track 289.9 -> 290.9 mm
