File: CAD/Methanesense/Methanesense.kicad_sch (KiCad schematic)
At the start: 23 parts, among them J2 SM12B-GHS-TB(LF)(SN), U2 ADS1115IDGS, U5 MCP4725xxx-xCH

Commit message: WIP
Parts:
- removed C13, C14, C15, C16, C17, C18: 0.1uF, Capacitor_SMD:C_0402_1005Metric, symbol Library:C
- removed C19, C20: 1uF, Capacitor_SMD:C_0402_1005Metric, symbol Library:C
- removed D1, D2, D3: 1N5819WS, Diode_SMD:D_SOD-323, symbol Library:1N4148WS
- removed J2: SM12B-GHS-TB(LF)(SN), Connector_JST:JST_GH_SM12B-GHS-TB_1x12-1MP_P1.25mm_Horizontal, symbol Library:Conn_01x14_Pin
- removed R10, R11, R8, R9: 499R, Resistor_SMD:R_0402_1005Metric, symbol Library:R
- removed R12, R3, R6: 10K, Resistor_SMD:R_0402_1005Metric, symbol Library:R
- removed R13: 100R, Resistor_SMD:R_0402_1005Metric, symbol Library:R
- removed R7: 309k, Resistor_SMD:R_0402_1005Metric, symbol Library:R
- removed U2: ADS1115IDGS, Package_SO:TSSOP-10_3x3mm_P0.5mm, symbol Analog_ADC:ADS1115IDGS
- removed U5: MCP4725xxx-xCH, Package_TO_SOT_SMD:SOT-23-6, symbol Analog_DAC:MCP4725xxx-xCH
Other:
- added sheet ENV_SENSOR (ENV_SENSOR.kicad_sch)
- added sheet GAS_SENSOR (GAS_SENSOR.kicad_sch)
- sheet POWER ports: added RXD, SCL, SDA, TXD, ~{CTS}, ~{RTS}; removed none
- sheet nrf9160 ports: added BUS; removed none
- note removed: "ADC"
- note removed: "Addr: 1001000"
- note removed: "Addr: 1100001"
- note removed: "DAC"
- note removed: "Output connector"
- note removed: "Voltage Monitor"

Commit message: Allmost there
Other:
- sheet POWER ports: added USB_DET; removed none
Changed lines of the file:
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@@
+	)
+	(bus_entry
+		(at 137.16 58.42)
+		(size 2.54 -2.54)
+		(stroke
+			(width 0)
+			(type default)
+		)
 	)
 	(bus_entry
@@
 		)
 	)
+	(bus
+		(pts
+			(xy 139.7 55.88) (xy 139.7 62.23)
+		)
+		(stroke
+			(width 0)
+			(type default)
+		)
+	)
 	(wire
 		(pts
@@
 	(bus
 		(pts
-			(xy 139.7 53.34) (xy 139.7 62.23)
+			(xy 139.7 53.34) (xy 139.7 55.88)
 		)
 		(stroke
@@
 		(pts
 			(xy 124.46 50.8) (xy 137.16 50.8)
+		)
+		(stroke
+			(width 0)
+			(type default)
+		)
+	)
+	(wire
+		(pts
+			(xy 124.46 58.42) (xy 137.16 58.42)
 		)
 		(stroke
@@
 			(effects
 				(font
+					(size 1.27 1.27)
+				)
+				(justify right)
+			)
+		)
+		(pin "USB_DET" input
+			(at 124.46 58.42 0)
+			(effects
+				(font

Commit message: WIP
Other:
- sheet GAS_SENSOR ports: added NRF_AIN0, NRF_AIN1; removed AIN0, AIN1
- sheet nrf9160 ports: added ADC_DRDY, AIN0, AIN1, Heater, RXD, SCL, SDA, Sensor, TXD, USB_DET, ~{CTS}, ~{RTS}; removed BUS

Commit message: Rev 2.0.0
Changed lines of the file:
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@@
+	(wire
+		(pts
+			(xy 124.46 96.52) (xy 132.08 96.52)
+		)
+		(stroke
+			(width 0)
+			(type default)
+		)
+	)
 	(wire
 		(pts
@@
 		(pts
 			(xy 124.46 114.3) (xy 137.16 114.3)
-		)
-		(stroke
-			(width 0)
-			(type default)
-		)
-	)
-	(wire
-		(pts
-			(xy 124.46 96.52) (xy 137.16 96.52)
 		)
 		(stroke
@@
 	(wire
 		(pts
-			(xy 124.46 99.06) (xy 137.16 99.06)
+			(xy 124.46 99.06) (xy 132.08 99.06)
 		)
 		(stroke

Commit message: rev 1.2
Other:
- sheet GAS_SENSOR ports: added AIN2, AIN3; removed NRF_AIN0, NRF_AIN1
- sheet POWER ports: added AI1, AI2, AIO1, AIO2, IRQ0, IRQ1, OD1, OD2; removed RXD, TXD, ~{CTS}, ~{RTS}
- sheet nrf9160 ports: added AIO1, AIO2, IRQ0, IRQ1, OD1, OD2; removed AIN0, AIN1, RXD, TXD, ~{CTS}, ~{RTS}

Commit message: Feat: Rev 1.3
Parts:
- added H1, H2: MountingHole, MountingHole:MountingHole_2.2mm_M2, symbol Mechanical:MountingHole
Changed lines of the file:
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@@
+		)
+	)
+	(symbol
+		(lib_id "Mechanical:MountingHole")
+		(at 259.08 38.1 0)
+		(unit 1)
+		(exclude_from_sim yes)
+		(in_bom no)
+		(on_board yes)
+		(dnp no)
+		(fields_autoplaced yes)
+		(property "Reference" "H2"
+			(at 261.62 36.8299 0)
+			(effects
+				(font
+					(size 1.27 1.27)
+				)
+				(justify left)
+			)
+		)
+		(property "Value" "MountingHole"
+			(at 261.62 39.3699 0)
+			(effects
+				(font
+					(size 1.27 1.27)
+				)
+				(justify left)
+			)
+		)
+		(property "Footprint" "MountingHole:MountingHole_2.2mm_M2"
+			(at 259.08 38.1 0)
+			(effects
+				(font
+					(size 1.27 1.27)
+				)
+				(hide yes)
+			)
+		)
+		(property "Datasheet" "~"
+			(at 259.08 38.1 0)
+			(effects
+				(font
+					(size 1.27 1.27)
+				)
+				(hide yes)
+			)
+		)
+		(property "Description" "Mounting Hole without connection"
+			(at 259.08 38.1 0)
+			(effects
+				(font
+					(size 1.27 1.27)
+				)
+				(hide yes)
+			)
+		)
+		(property "TEST" ""
+			(at 259.08 38.1 0)
+			(effects
+				(font
+					(size 1.27 1.27)
+				)
+			)
+		)
+		(instances
+			(project ""
+				(path "/51bbc301-ea4a-44e0-84a7-cf42c64443ca"
+					(reference "H2")
+					(unit 1)
+				)
+			)
+		)
+	)
+	(symbol
+		(lib_id "Mechanical:MountingHole")
+		(at 259.08 27.94 0)
+		(unit 1)
+		(exclude_from_sim yes)
+		(in_bom no)
+		(on_board yes)
+		(dnp no)
+		(fields_autoplaced yes)
+		(property "Reference" "H1"
+			(at 261.62 26.6699 0)
+			(effects
+				(font
+					(size 1.27 1.27)
+				)
+				(justify left)
+			)
+		)
+		(property "Value" "MountingHole"
+			(at 261.62 29.2099 0)
+			(effects
+				(font
+					(size 1.27 1.27)
+				)
+				(justify left)
+			)
+		)
+		(property "Footprint" "MountingHole:MountingHole_2.2mm_M2"
+			(at 259.08 27.94 0)
+			(effects
+				(font
+					(size 1.27 1.27)
+				)
+				(hide yes)
+			)
+		)
+		(property "Datasheet" "~"
+			(at 259.08 27.94 0)
+			(effects
+				(font
+					(size 1.27 1.27)
+				)
+				(hide yes)
+			)
+		)
+		(property "Description" "Mounting Hole without connection"
+			(at 259.08 27.94 0)
+			(effects
+				(font
+					(size 1.27 1.27)
+				)
+				(hide yes)
+			)
+		)
+		(property "TEST" ""
+			(at 259.08 27.94 0)
+			(effects
+				(font
+					(size 1.27 1.27)
+				)
+			)
+		)
+		(instances
+			(project ""
+				(path "/51bbc301-ea4a-44e0-84a7-cf42c64443ca"
+					(reference "H1")
+					(unit 1)
+				)
+			)
 		)
 	)
