File: CAD/Methanesense/GAS_SENSOR.kicad_sch (KiCad schematic)
At the start: 21 parts, among them Q1 FDS6892A, U2 ADS1115IDGS

Commit message: Allmost there
Parts:
- removed C15, C16: 0.1uF, Capacitor_SMD:C_0603_1608Metric, symbol Library:C
- removed C18: 1uF, Capacitor_SMD:C_0603_1608Metric, symbol Library:C
- removed R4, R5: 499R, Resistor_SMD:R_0402_1005Metric, symbol Library:R
- removed R6: 10K, Resistor_SMD:R_0603_1608Metric, symbol Library:R
- R2, R3: footprint Resistor_SMD:R_0402_1005Metric -> Resistor_SMD:R_0603_1608Metric
- R7, R8: value 499R -> 0R; footprint Resistor_SMD:R_0402_1005Metric -> Resistor_SMD:R_0603_1608Metric
Connections:
- net AIN0: now also Q1.7 (D1), Q1.8 (D1), R9.1; no longer R7.1, R7.2, R9.2, S1.2 (Rs-)
- net AIN1: now also R9.2, S1.2 (Rs-); no longer Q1.5 (D2), Q1.6 (D2), R8.1, R8.2, R9.1
- net AIN2: now also U2.6 (AIN2)
- net AIN3: now also U2.7 (AIN3)
- net AIN1_: now reaches C14.2, C17.2, R3.1, U2.5 (AIN1)
- net AIN1_: now also R8.1
- net AIN0_: now reaches C13.2, C17.1, R2.1, U2.4 (AIN0)
- net AIN0_: now also R7.2
- net +2V0 renamed +2V0SW
- new net: Q1.5 (D2), Q1.6 (D2), S1.1 (Rh-)
- new net NRF_AIN0: R7.1
- new net NRF_AIN1: R8.2
Other:
- note added: "Addr: 100 1000"
- note removed: "Addr: 1001000"
- moved on the sheet: Q1A, Q1B, R10, R11, R7, R8

Commit message: WIP
Parts:
- S1: MPN (none) -> TGS8410
- U2: MPN (none) -> ADS1115IDGS
Changed lines of the file:
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@@
+			)
+		)
+		(property "MPN" ""
+			(at 57.15 109.22 0)
+			(effects
+				(font
+					(size 1.27 1.27)
+				)
+				(hide yes)
 			)
 		)
@@
 			)
 		)
+		(property "MPN" ""
+			(at 176.53 85.09 0)
+			(effects
+				(font
+					(size 1.27 1.27)
+				)
+				(hide yes)
+			)
+		)
 		(pin "1"
 		)
@@
 			)
 		)
+		(property "MPN" ""
+			(at 190.5 69.85 0)
+			(effects
+				(font
+					(size 1.27 1.27)
+				)
+				(hide yes)
+			)
+		)
 		(pin "1"
 		)
@@
 					(size 1.27 1.27)
 				)
+			)
+		)
+		(property "MPN" ""
+			(at 82.55 109.22 0)
+			(effects
+				(font
+					(size 1.27 1.27)
+				)
+				(hide yes)
 			)
 		)
@@
 			)
 		)
+		(property "MPN" ""
+			(at 187.96 77.47 0)
+			(effects
+				(font
+					(size 1.27 1.27)
+				)
+				(hide yes)
+			)
+		)
 		(pin "1"
 		)
@@
 			)
 		)
+		(property "MPN" ""
+			(at 217.17 118.11 0)
+			(effects
+				(font
+					(size 1.27 1.27)
+				)
+				(hide yes)
+			)
+		)
 		(pin "1"
 		)
@@
 			)
 		)
+		(property "MPN" ""
+			(at 76.2 113.03 0)
+			(effects
+				(font
+					(size 1.27 1.27)
+				)
+				(hide yes)
+			)
+		)
 		(pin "1"
 		)
@@
 			)
 		)
+		(property "MPN" "ADS1115IDGS"
+			(at 217.17 88.9 0)
+			(effects
+				(font
+					(size 1.27 1.27)
+				)
+				(hide yes)
+			)
+		)
 		(pin "1"
 		)
@@
 					(size 1.27 1.27)
 				)
+			)
+		)
+		(property "MPN" ""
+			(at 167.64 73.66 0)
+			(effects
+				(font
+					(size 1.27 1.27)
+				)
+				(hide yes)
 			)
 		)
@@
 			)
 		)
+		(property "MPN" ""
+			(at 85.09 97.79 0)
+			(effects
+				(font
+					(size 1.27 1.27)
+				)
+				(hide yes)
+			)
+		)
 		(pin "1"
 		)
@@
 			)
 		)
+		(property "MPN" ""
+			(at 227.33 118.11 0)
+			(effects
+				(font
+					(size 1.27 1.27)
+				)
+				(hide yes)
+			)
+		)
 		(pin "1"
 		)
@@
 			)
 		)
+		(property "MPN" ""
+			(at 50.8 113.03 0)
+			(effects
+				(font
+					(size 1.27 1.27)
+				)
+				(hide yes)
+			)
+		)
 		(pin "1"
 		)
@@
 		)
 		(property "LCSC Part #" "C307331"
+			(at 176.53 69.85 0)
+			(effects
+				(font
+					(size 1.27 1.27)
+				)
+				(hide yes)
+			)
+		)
+		(property "MPN" ""
 			(at 176.53 69.85 0)
 			(effects
@@
 			)
 		)
+		(property "MPN" "TGS8410"
+			(at 71.12 81.28 0)
+			(effects
+				(font
+					(size 1.27 1.27)
+				)
+				(hide yes)
+			)
+		)
 		(pin "3"
 		)
@@
 			)
 		)
+		(property "MPN" ""
+			(at 167.64 81.28 0)
+			(effects
+				(font
+					(size 1.27 1.27)
+				)
+				(hide yes)
+			)
+		)
 		(pin "1"
 		)
@@
 			)
 		)
+		(property "MPN" ""
+			(at 190.5 85.09 0)
+			(effects
+				(font
+					(size 1.27 1.27)
+				)
+				(hide yes)
+			)
+		)

Commit message: NRF footprint change
Parts:
- C13, C14, C17, C19, C20: LCSC Part # C307331 -> (none)
- Q1: value FDS6892A -> FDS6898A; MPN (none) -> FDS6898A
- R2, R3: value 499R -> 470R; LCSC Part # C25076 -> (none)
- R7, R8: LCSC Part # C25076 -> (none)
- S1: now not fitted
Changed lines of the file:
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@@
 			)
 		)
-		(property "Value" "FDS6892A"
+		(property "Value" "FDS6898A"
 			(at 60.96 112.268 0)
 			(effects
@@
 			)
 		)
-		(property "Description" "4.8A Id, 20V Vds, Dual N-Channel MOSFET , 37mOhm Ron, SO-8"
+		(property "Description" "9.4A Id, 20V Vds, Dual N-Channel MOSFET , 14mOhm Ron, SO-8"
 			(at 57.15 109.22 0)
 			(effects
@@
 			)
 		)
-		(property "MPN" ""
+		(property "MPN" "FDS6898A"
 			(at 57.15 109.22 0)
 			(effects
@@
 			)
 		)
-		(property "Description" ""
-			(at 176.53 85.09 0)
-			(effects
-				(font
-					(size 1.27 1.27)
-				)
-				(hide yes)
-			)
-		)
-		(property "LCSC Part #" "C307331"
-			(at 176.53 85.09 0)
-			(effects
-				(font
-					(size 1.27 1.27)
-				)
-				(hide yes)
-			)
-		)
-		(property "MPN" ""
+		(property "Description" "Unpolarized capacitor"
 			(at 176.53 85.09 0)
 			(effects
@@
 			)
 		)
-		(property "LCSC Part #" "C25076"
-			(at 190.5 69.85 0)
-			(effects
-				(font
-					(size 1.27 1.27)
-				)
-				(hide yes)
-			)
-		)
 		(property "TEST" ""
 			(at 190.5 69.85 0)
@@
 			)
 		)
-		(property "MPN" ""
-			(at 190.5 69.85 0)
-			(effects
-				(font
-					(size 1.27 1.27)
-				)
-				(hide yes)
-			)
-		)
 		(pin "1"
 		)
@@
 			)
 		)
-		(property "Value" "FDS6892A"
+		(property "Value" "FDS6898A"
 			(at 86.614 111.76 0)
 			(effects
@@
 			)
 		)
-		(property "Description" "4.8A Id, 20V Vds, Dual N-Channel MOSFET , 37mOhm Ron, SO-8"
+		(property "Description" "9.4A Id, 20V Vds, Dual N-Channel MOSFET , 14mOhm Ron, SO-8"
 			(at 82.55 109.22 0)
 			(effects
@@
 			)
 		)
-		(property "MPN" ""
+		(property "MPN" "FDS6898A"
 			(at 82.55 109.22 0)
 			(effects
@@
 			)
 		)
-		(property "Description" ""
-			(at 187.96 77.47 0)
-			(effects
-				(font
-					(size 1.27 1.27)
-				)
-				(hide yes)
-			)
-		)
-		(property "LCSC Part #" "C307331"
+		(property "Description" "Unpolarized capacitor"
 			(at 187.96 77.47 0)
 			(effects
@@
 					(size 1.27 1.27)
 				)
-			)
-		)
-		(property "MPN" ""
-			(at 187.96 77.47 0)
-			(effects
-				(font
-					(size 1.27 1.27)
-				)
-				(hide yes)
 			)
 		)
@@
 			)
 		)
-		(property "Description" ""
-			(at 217.17 118.11 0)
-			(effects
-				(font
-					(size 1.27 1.27)
-				)
-				(hide yes)
-			)
-		)
-		(property "LCSC Part #" "C307331"
-			(at 217.17 118.11 0)
-			(effects
-				(font
-					(size 1.27 1.27)
-				)
-				(hide yes)
-			)
-		)
-		(property "MPN" ""
+		(property "Description" "Unpolarized capacitor"
 			(at 217.17 118.11 0)
 			(effects
@@
 			)
 		)
-		(property "MPN" ""
-			(at 76.2 113.03 0)
-			(effects
-				(font
-					(size 1.27 1.27)
-				)
-				(hide yes)
-			)
-		)
 		(pin "1"
 		)
@@
 			)
 		)
-		(property "Value" "499R"
+		(property "Value" "470R"
 			(at 165.1 73.66 90)
 			(effects
@@
 			)
 		)
-		(property "LCSC Part #" "C25076"
-			(at 167.64 73.66 0)
-			(effects
-				(font
-					(size 1.27 1.27)
-				)
-				(hide yes)
-			)
-		)
 		(property "TEST" ""
 			(at 167.64 73.66 0)
@@
 					(size 1.27 1.27)
 				)
-			)
-		)
-		(property "MPN" ""
-			(at 167.64 73.66 0)
-			(effects
-				(font
-					(size 1.27 1.27)
-				)
-				(hide yes)
 			)
 		)
@@
 			)
 		)
-		(property "LCSC Part #" ""
-			(at 85.09 97.79 0)
-			(effects
-				(font
-					(size 1.27 1.27)
-				)
-				(hide yes)
-			)
-		)
 		(property "TEST" ""
 			(at 85.09 97.79 0)
@@
 					(size 1.27 1.27)
 				)
-			)
-		)
-		(property "MPN" ""
-			(at 85.09 97.79 0)
-			(effects
-				(font
-					(size 1.27 1.27)
-				)
-				(hide yes)
 			)
 		)
@@
 			)
 		)
-		(property "Description" ""
-			(at 227.33 118.11 0)
-			(effects
-				(font
-					(size 1.27 1.27)
-				)
-				(hide yes)
-			)
-		)
-		(property "LCSC Part #" "C307331"
+		(property "Description" "Unpolarized capacitor"
 			(at 227.33 118.11 0)
 			(effects
@@
 					(size 1.27 1.27)
 				)
-			)
-		)
-		(property "MPN" ""
-			(at 227.33 118.11 0)
-			(effects
-				(font
-					(size 1.27 1.27)
-				)
-				(hide yes)
 			)
 		)
@@
 			)
 		)
-		(property "MPN" ""
-			(at 50.8 113.03 0)
-			(effects
-				(font
-					(size 1.27 1.27)
-				)
-				(hide yes)
-			)
-		)
 		(pin "1"
 		)
@@
 			)
 		)
-		(property "Description" ""
-			(at 176.53 69.85 0)
-			(effects
-				(font
-					(size 1.27 1.27)
-				)
-				(hide yes)
-			)
-		)
-		(property "LCSC Part #" "C307331"
-			(at 176.53 69.85 0)
-			(effects
-				(font
-					(size 1.27 1.27)
-				)
-				(hide yes)
-			)
-		)
-		(property "MPN" ""
+		(property "Description" "Unpolarized capacitor"
 			(at 176.53 69.85 0)
 			(effects
@@
 		(in_bom yes)
 		(on_board yes)
-		(dnp no)
+		(dnp yes)
 		(fields_autoplaced yes)
 		(property "Reference" "S1"
@@
 			)
 		)
+		(property "TEST" ""
+			(at 71.12 81.28 0)
+			(effects
+				(font
+					(size 1.27 1.27)
+				)
+			)
+		)
 		(property "MPN" "TGS8410"
 			(at 71.12 81.28 0)
@@
 			)
 		)
-		(property "Value" "499R"
+		(property "Value" "470R"
 			(at 165.1 81.28 90)
 			(effects
@@
 			)
 		)
-		(property "LCSC Part #" "C25076"
-			(at 167.64 81.28 0)
-			(effects
-				(font
-					(size 1.27 1.27)
-				)
-				(hide yes)
-			)
-		)
 		(property "TEST" ""
 			(at 167.64 81.28 0)
@@
 					(size 1.27 1.27)
 				)
-			)
-		)
-		(property "MPN" ""
-			(at 167.64 81.28 0)
-			(effects
-				(font
-					(size 1.27 1.27)
-				)
-				(hide yes)
 			)
 		)
@@
 			)
 		)
-		(property "LCSC Part #" "C25076"
-			(at 190.5 85.09 0)
-			(effects
-				(font
-					(size 1.27 1.27)
-				)
-				(hide yes)
-			)
-		)
 		(property "TEST" ""
 			(at 190.5 85.09 0)
@@
 			)
 		)
-		(property "MPN" ""
-			(at 190.5 85.09 0)
-			(effects
-				(font
-					(size 1.27 1.27)
-				)
-				(hide yes)
-			)
-		)

Commit message: Rev 2.0.0
Parts:
- S1: now fitted
Changed lines of the file:
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@@
 			)
 		)
-		(property "Description" ""
+		(property "Description" "Resistor"
 			(at 190.5 69.85 0)
 			(effects
@@
 			)
 		)
-		(property "Description" ""
+		(property "Description" "Resistor"
 			(at 167.64 73.66 0)
 			(effects
@@
 			)
 		)
-		(property "Description" ""
+		(property "Description" "Resistor"
 			(at 85.09 97.79 0)
 			(effects
@@
 		(in_bom yes)
 		(on_board yes)
-		(dnp yes)
+		(dnp no)
 		(fields_autoplaced yes)
 		(property "Reference" "S1"
@@
 			)
 		)
-		(property "Description" ""
+		(property "Description" "Resistor"
 			(at 167.64 81.28 0)
 			(effects
@@
 			)
 		)
-		(property "Description" ""
+		(property "Description" "Resistor"
 			(at 190.5 85.09 0)
 			(effects

Commit message: rev 1.2
Parts:
- removed C19: 0.1uF, Capacitor_SMD:C_0603_1608Metric, symbol Library:C
- removed R7, R8: 0R, Resistor_SMD:R_0603_1608Metric, symbol Library:R
- added C1, C2: 0.1uF, Capacitor_SMD:C_0603_1608Metric, symbol Library:C
- added R12, R5: 470R, Resistor_SMD:R_0603_1608Metric, symbol Library:R
- R9: value <2k -> 12k; now fitted
Connections:
- net AIN2: now also R5.2; no longer U2.6 (AIN2)
- net AIN3: now also R12.2; no longer U2.7 (AIN3)
- net GND: now also C1.1, C2.1
- net +2V0SW renamed +2V0
- new net AIN2_: C1.2, R5.1, U2.6 (AIN2)
- new net AIN3_: C2.2, R12.1, U2.7 (AIN3)
Other:
- note added: "Addr: 100 1000 hex 0x48"
- note removed: "Addr: 100 1000"

Commit message: Feat: Rev 1.3
Parts:
- added TP11: AIN1, TestPoint:TestPoint_Pad_D1.0mm, symbol Connector:TestPoint
- added TP12: AIN0, TestPoint:TestPoint_Pad_D1.0mm, symbol Connector:TestPoint
- added TP13: SEN, TestPoint:TestPoint_Pad_D1.0mm, symbol Connector:TestPoint
- added TP14: HEAT, TestPoint:TestPoint_Pad_D1.0mm, symbol Connector:TestPoint
- added TP18: GND, TestPoint:TestPoint_Pad_D1.0mm, symbol Connector:TestPoint
- U2: value ADS1115IDGS -> ADS1115IDGST; MPN ADS1115IDGS -> ADS1115IDGSR
Connections:
- net AIN0: now also TP12.1
- net AIN1: now also TP11.1
- net GND: now also TP18.1
- net Heater: now also TP14.1
- net Sensor: now also TP13.1
Other:
- title: (none) -> GAS SENSOR

Commit message: Feat: Prettified repo Readme
Connections:
- net Heater: now also Q1.4 (G2), R10.2, TP13.1; no longer Q1.2 (G1), R11.2, TP14.1
- net Sensor: now also Q1.2 (G1), R11.2, TP14.1; no longer Q1.4 (G2), R10.2, TP13.1
Changed lines of the file:
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@@
 	(hierarchical_label "Sensor"
 		(shape input)
-		(at 44.45 109.22 180)
+		(at 71.12 109.22 180)
 		(effects
 			(font
@@
 	(hierarchical_label "Heater"
 		(shape input)
-		(at 71.12 109.22 180)
+		(at 44.45 109.22 180)
 		(effects
 			(font
