File: CAD/Methanesense/nrf9160.kicad_sch (KiCad schematic)
At the start: 48 parts, among them J1 HIROSE ELECTRIC U.FL-R-SMT-1, J3 693043020611, J4 HIROSE ELECTRIC U.FL-R-SMT-1, J5 Conn_01x13_Pin, J6 JLINK, Q2 FDS6898A, SW1 KMR223NGLFG, U5 nRF9160-SICA, U8 USBLC6-4SC6, U9 TPS22917DBV

Commit message: Feat: Prettified repo Readme
Parts:
- AE1: value ~ -> 2361492-1; MPN (none) -> 2361492-1
Changed lines of the file:
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@@
 	(hierarchical_label "Heater"
 		(shape input)
-		(at 33.02 59.69 180)
+		(at 33.02 57.15 180)
 		(effects
 			(font
@@
 	(hierarchical_label "Sensor"
 		(shape input)
-		(at 33.02 57.15 180)
+		(at 33.02 59.69 180)
 		(effects
 			(font
@@
 			)
 		)
-		(property "Value" "~"
-			(at 259.334 57.658 0)
+		(property "Value" "2361492-1"
+			(at 261.366 56.896 0)
 			(effects
 				(font
@@
 			)
 		)
+		(property "MPN" "2361492-1"
+			(at 259.08 54.61 0)
+			(effects
+				(font
+					(size 1.27 1.27)
+				)
+				(hide yes)
+			)
+		)
